Commit message: moveit config ws

File: ws/tg2_ws/src/tg2_description/urdf/tiangong2_EVT_V2.urdf (robot description, URDF)
Before this commit: robot humanoid, 31 links, 30 joints
Links:
- added link base
- link ankle_pitch_l_link: geometry collision mesh filename=package://tg2_description/urdf/meshes/ankle_pitch_l_link.STL; visual mesh filename=package://tg2_description/urdf/meshes/ankle_pitch_l_link.STL
- link ankle_pitch_r_link: geometry collision mesh filename=package://tg2_description/urdf/meshes/ankle_pitch_r_link.STL; visual mesh filename=package://tg2_description/urdf/meshes/ankle_pitch_r_link.STL
- link ankle_roll_l_link: geometry collision mesh filename=package://tg2_description/urdf/meshes/ankle_roll_l_link.STL; visual mesh filename=package://tg2_description/urdf/meshes/ankle_roll_l_link.STL
- link ankle_roll_r_link: geometry collision mesh filename=package://tg2_description/urdf/meshes/ankle_roll_r_link.STL; visual mesh filename=package://tg2_description/urdf/meshes/ankle_roll_r_link.STL
- link elbow_pitch_l_link: geometry collision mesh filename=package://tg2_description/urdf/meshes/elbow_pitch_l_link.STL; visual mesh filename=package://tg2_description/urdf/meshes/elbow_pitch_l_link.STL
- link elbow_pitch_r_link: geometry collision mesh filename=package://tg2_description/urdf/meshes/elbow_pitch_r_link.STL; visual mesh filename=package://tg2_description/urdf/meshes/elbow_pitch_r_link.STL
- link elbow_yaw_l_link: geometry collision mesh filename=package://tg2_description/urdf/meshes/elbow_yaw_l_link.STL; visual mesh filename=package://tg2_description/urdf/meshes/elbow_yaw_l_link.STL
- link elbow_yaw_r_link: geometry collision mesh filename=package://tg2_description/urdf/meshes/elbow_yaw_r_link.STL; visual mesh filename=package://tg2_description/urdf/meshes/elbow_yaw_r_link.STL
- link head_pitch_link: geometry collision mesh filename=package://tg2_description/urdf/meshes/head_pitch_link.STL; visual mesh filename=package://tg2_description/urdf/meshes/head_pitch_link.STL
- link head_roll_link: geometry collision mesh filename=package://tg2_description/urdf/meshes/head_roll_link.STL; visual mesh filename=package://tg2_description/urdf/meshes/head_roll_link.STL
- link head_yaw_link: geometry collision mesh filename=package://tg2_description/urdf/meshes/head_yaw_link.STL; visual mesh filename=package://tg2_description/urdf/meshes/head_yaw_link.STL
- link hip_pitch_l_link: geometry collision mesh filename=package://tg2_description/urdf/meshes/hip_pitch_l_link.STL; visual mesh filename=package://tg2_description/urdf/meshes/hip_pitch_l_link.STL
- link hip_pitch_r_link: geometry collision mesh filename=package://tg2_description/urdf/meshes/hip_pitch_r_link.STL; visual mesh filename=package://tg2_description/urdf/meshes/hip_pitch_r_link.STL
- link hip_roll_l_link: geometry collision mesh filename=package://tg2_description/urdf/meshes/hip_roll_l_link.STL; visual mesh filename=package://tg2_description/urdf/meshes/hip_roll_l_link.STL
- link hip_roll_r_link: geometry collision mesh filename=package://tg2_description/urdf/meshes/hip_roll_r_link.STL; visual mesh filename=package://tg2_description/urdf/meshes/hip_roll_r_link.STL
- link hip_yaw_l_link: geometry collision mesh filename=package://tg2_description/urdf/meshes/hip_yaw_l_link.STL; visual mesh filename=package://tg2_description/urdf/meshes/hip_yaw_l_link.STL
- link hip_yaw_r_link: geometry collision mesh filename=package://tg2_description/urdf/meshes/hip_yaw_r_link.STL; visual mesh filename=package://tg2_description/urdf/meshes/hip_yaw_r_link.STL
- link knee_pitch_l_link: geometry collision mesh filename=package://tg2_description/urdf/meshes/knee_pitch_l_link.STL; visual mesh filename=package://tg2_description/urdf/meshes/knee_pitch_l_link.STL
- link knee_pitch_r_link: geometry collision mesh filename=package://tg2_description/urdf/meshes/knee_pitch_r_link.STL; visual mesh filename=package://tg2_description/urdf/meshes/knee_pitch_r_link.STL
- link pelvis: geometry collision mesh filename=package://tg2_description/urdf/meshes/pelvis.STL; visual mesh filename=package://tg2_description/urdf/meshes/pelvis.STL
- link shoulder_pitch_l_link: geometry collision mesh filename=package://tg2_description/urdf/meshes/shoulder_pitch_l_link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; visual mesh filename=package://tg2_description/urdf/meshes/shoulder_pitch_l_link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
- link shoulder_pitch_r_link: geometry collision mesh filename=package://tg2_description/urdf/meshes/shoulder_pitch_r_link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; visual mesh filename=package://tg2_description/urdf/meshes/shoulder_pitch_r_link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
- link shoulder_roll_l_link: geometry collision mesh filename=package://tg2_description/urdf/meshes/shoulder_roll_l_link.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; visual mesh filename=package://tg2_description/urdf/meshes/shoulder_roll_l_link.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
- link shoulder_roll_r_link: geometry collision mesh filename=package://tg2_description/urdf/meshes/shoulder_roll_r_link.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; visual mesh filename=package://tg2_description/urdf/meshes/shoulder_roll_r_link.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
- link shoulder_yaw_l_link: geometry collision mesh filename=package://tg2_description/urdf/meshes/shoulder_yaw_l_link.S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; visual mesh filename=package://tg2_description/urdf/meshes/shoulder_yaw_l_link.S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
- link shoulder_yaw_r_link: geometry collision mesh filename=package://tg2_description/urdf/meshes/shoulder_yaw_r_link.S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; visual mesh filename=package://tg2_description/urdf/meshes/shoulder_yaw_r_link.S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
- link waist_yaw_link: geometry collision mesh filename=package://tg2_description/urdf/meshes/waist_yaw_link.STL; visual mesh filename=package://tg2_description/urdf/meshes/waist_yaw_link.STL
- link wrist_pitch_l_link: geometry collision mesh filename=package://tg2_description/urdf/meshes/wrist_pitch_l_link.STL; visual mesh filename=package://tg2_description/urdf/meshes/wrist_pitch_l_link.STL
- link wrist_pitch_r_link: geometry collision mesh filename=package://tg2_description/urdf/meshes/wrist_pitch_r_link.STL; visual mesh filename=package://tg2_description/urdf/meshes/wrist_pitch_r_link.STL
- link wrist_roll_l_link: geometry collision mesh filename=package://tg2_description/urdf/meshes/wrist_roll_l_link.STL; visual mesh filename=package://tg2_description/urdf/meshes/wrist_roll_l_link.STL
- link wrist_roll_r_link: geometry collision mesh filename=package://tg2_description/urdf/meshes/wrist_roll_r_link.STL; visual mesh filename=package://tg2_description/urdf/meshes/wrist_roll_r_link.STL
Joints:
- added joint base_to_pelvis: type fixed, parent base, child pelvis, origin xyz=0 0 0 rpy=0 0 0

Commit message: clean up codebase

File: ws/tg2_ws/src/tg2_description/urdf/tiangong2_EVT_V2.urdf (robot description, URDF)
Before this commit: robot humanoid, 32 links, 31 joints
Links:
- link ankle_pitch_l_link: geometry collision mesh filename=package://tg2_description/urdf/meshes_collision/ankle_pitch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; visual mesh filename=package://tg2_description/urdf/meshes/ankle_pitch_l_link.STL
- link ankle_pitch_r_link: geometry collision mesh filename=package://tg2_description/urdf/meshes_collision/ankle_pitch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; visual mesh filename=package://tg2_description/urdf/meshes/ankle_pitch_r_link.STL
- link ankle_roll_l_link: geometry collision mesh filename=package://tg2_description/urdf/meshes_collision/ankle_roll_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; visual mesh filename=package://tg2_description/urdf/meshes/ankle_roll_l_link.STL
- link ankle_roll_r_link: geometry collision mesh filename=package://tg2_description/urdf/meshes_collision/ankle_roll_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; visual mesh filename=package://tg2_description/urdf/meshes/ankle_roll_r_link.STL
- link elbow_pitch_l_link: geometry collision mesh filename=package://tg2_description/urdf/meshes_collision/elbow_pitch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; visual mesh filename=package://tg2_description/urdf/meshes/elbow_pitch_l_link.STL
- link elbow_pitch_r_link: geometry collision mesh filename=package://tg2_description/urdf/meshes_collision/elbow_pitch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; visual mesh filename=package://tg2_description/urdf/meshes/elbow_pitch_r_link.STL
- link elbow_yaw_l_link: geometry collision mesh filename=package://tg2_description/urdf/meshes_collision/elbow_yaw_l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; visual mesh filename=package://tg2_description/urdf/meshes/elbow_yaw_l_link.STL
- link elbow_yaw_r_link: geometry collision mesh filename=package://tg2_description/urdf/meshes_collision/elbow_yaw_r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; visual mesh filename=package://tg2_description/urdf/meshes/elbow_yaw_r_link.STL
- link head_pitch_link: geometry collision mesh filename=package://tg2_description/urdf/meshes_collision/head_pitch_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; visual mesh filename=package://tg2_description/urdf/meshes/head_pitch_link.STL
- link head_roll_link: geometry collision mesh filename=package://tg2_description/urdf/meshes_collision/head_roll_l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; visual mesh filename=package://tg2_description/urdf/meshes/head_roll_link.STL
- link head_yaw_link: geometry collision mesh filename=package://tg2_description/urdf/meshes_collision/head_yaw_li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; visual mesh filename=package://tg2_description/urdf/meshes/head_yaw_link.STL
- link hip_pitch_l_link: geometry collision mesh filename=package://tg2_description/urdf/meshes_collision/hip_pitch_l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; visual mesh filename=package://tg2_description/urdf/meshes/hip_pitch_l_link.STL
- link hip_pitch_r_link: geometry collision mesh filename=package://tg2_description/urdf/meshes_collision/hip_pitch_r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; visual mesh filename=package://tg2_description/urdf/meshes/hip_pitch_r_link.STL
- link hip_roll_l_link: geometry collision mesh filename=package://tg2_description/urdf/meshes_collision/hip_roll_l_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; visual mesh filename=package://tg2_description/urdf/meshes/hip_roll_l_link.STL
- link hip_roll_r_link: geometry collision mesh filename=package://tg2_description/urdf/meshes_collision/hip_roll_r_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; visual mesh filename=package://tg2_description/urdf/meshes/hip_roll_r_link.STL
- link hip_yaw_l_link: geometry collision mesh filename=package://tg2_description/urdf/meshes_collision/hip_yaw_l_l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; visual mesh filename=package://tg2_description/urdf/meshes/hip_yaw_l_link.STL
- link hip_yaw_r_link: geometry collision mesh filename=package://tg2_description/urdf/meshes_collision/hip_yaw_r_l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; visual mesh filename=package://tg2_description/urdf/meshes/hip_yaw_r_link.STL
- link knee_pitch_l_link: geometry collision mesh filename=package://tg2_description/urdf/meshes_collision/knee_pitch_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; visual mesh filename=package://tg2_description/urdf/meshes/knee_pitch_l_link.STL
- link knee_pitch_r_link: geometry collision mesh filename=package://tg2_description/urdf/meshes_collision/knee_pitch_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; visual mesh filename=package://tg2_description/urdf/meshes/knee_pitch_r_link.STL
- link pelvis: geometry collision mesh filename=package://tg2_description/urdf/meshes_collision/pelvis.STL; visual mesh filename=package://tg2_description/urdf/meshes/pelvis.STL
- link shoulder_pitch_l_link: geometry collision mesh filename=package://tg2_description/urdf/meshes_collision/shoulder_pi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; visual mesh filename=package://tg2_description/urdf/meshes/shoulder_pitch_l_link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
- link shoulder_pitch_r_link: geometry collision mesh filename=package://tg2_description/urdf/meshes_collision/shoulder_pi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; visual mesh filename=package://tg2_description/urdf/meshes/shoulder_pitch_r_link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
- link shoulder_roll_l_link: geometry collision mesh filename=package://tg2_description/urdf/meshes_collision/shoulder_ro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; visual mesh filename=package://tg2_description/urdf/meshes/shoulder_roll_l_link.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
- link shoulder_roll_r_link: geometry collision mesh filename=package://tg2_description/urdf/meshes_collision/shoulder_ro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; visual mesh filename=package://tg2_description/urdf/meshes/shoulder_roll_r_link.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
- link shoulder_yaw_l_link: geometry collision mesh filename=package://tg2_description/urdf/meshes_collision/shoulder_ya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; visual mesh filename=package://tg2_description/urdf/meshes/shoulder_yaw_l_link.S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
- link shoulder_yaw_r_link: geometry collision mesh filename=package://tg2_description/urdf/meshes_collision/shoulder_ya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; visual mesh filename=package://tg2_description/urdf/meshes/shoulder_yaw_r_link.S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
- link waist_yaw_link: geometry collision mesh filename=package://tg2_description/urdf/meshes_collision/waist_yaw_l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; visual mesh filename=package://tg2_description/urdf/meshes/waist_yaw_link.STL
- link wrist_pitch_l_link: geometry collision mesh filename=package://tg2_description/urdf/meshes_collision/wrist_pitch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; visual mesh filename=package://tg2_description/urdf/meshes/wrist_pitch_l_link.STL
- link wrist_pitch_r_link: geometry collision mesh filename=package://tg2_description/urdf/meshes_collision/wrist_pitch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; visual mesh filename=package://tg2_description/urdf/meshes/wrist_pitch_r_link.STL
- link wrist_roll_l_link: geometry collision mesh filename=package://tg2_description/urdf/meshes_collision/wrist_roll_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; visual mesh filename=package://tg2_description/urdf/meshes/wrist_roll_l_link.STL
- link wrist_roll_r_link: geometry collision mesh filename=package://tg2_description/urdf/meshes_collision/wrist_roll_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; visual mesh filename=package://tg2_description/urdf/meshes/wrist_roll_r_link.STL
